File: Mini-BT-Pcb-328P.kicad_pcb (KiCad board)
At the start: 2 copper layers, 55 x 35 mm, 51 parts, among them J1 Analog IN, J2 USB_B_Micro, J5 ANT, J6 Booster, P1 MYSX_2.6, Q1 FDN338P, Q2 FDN337N, SW2 Reset, SW3 SW_Reed, U1 ME2188C33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

Commit message: routing test 2
Parts:
- removed J6: Booster, Connector_PinHeader_2.54mm:PinHeader_2x03_P2.54mm_Vertical_SMD
- added J3: Booster CE, Connector_PinHeader_2.54mm:PinHeader_2x03_P2.54mm_Vertical_SMD, F.Cu at (178.8, 102.4)
- C1: moved to F.Cu
- C11, R4, R5, SW2: moved to B.Cu
- moved R4 22.1 mm to (170.4, 78.7), turned to 180 degrees
- moved SW2 21.8 mm to (145.8, 82.0), turned to 0 degrees
- moved C1 21.8 mm to (163.8, 93.5), turned to 180 degrees
- moved R5 20.0 mm to (140.5, 78.0), turned to 90 degrees
- moved C11 19.4 mm to (143.1, 79.0), turned to 0 degrees
- moved C10 17.4 mm to (142.8, 74.9), turned to 180 degrees
- moved C8 17.3 mm to (147.1, 74.9), turned to 180 degrees
- moved R10 15.2 mm to (138.9, 96.3)
- moved C4 14.5 mm to (139.2, 86.9), turned to 90 degrees
- moved U2 14.4 mm to (135.4, 86.9), turned to 180 degrees
- moved R2 12.9 mm to (151.9, 84.3)
- moved U4 8.65 mm to (145.0, 81.3), turned to 270 degrees
- moved C7 8.20 mm to (144.3, 91.2), turned to 0 degrees
- moved R7 7.06 mm to (138.9, 91.9)
- moved C12 7.06 mm to (147.7, 76.7), turned to 180 degrees
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Routing:
- net VCC: track 81.3 -> 218.2 mm, vias 1 -> 14
- net RESET: track 110.6 -> 18.2 mm, vias 8 -> 3
- net D3: track 81.5 -> 0.00 mm, vias 3 -> 0
- net D2: track 125.1 -> 58.6 mm, vias 7 -> 6
- net D9: track 42.7 -> 91.3 mm, vias 3 -> 6
- net A3: track 75.7 -> 27.3 mm, vias 5 -> 2
- net D6: track 62.2 -> 27.0 mm, vias 4 -> 2
- net D5: track 57.5 -> 25.0 mm, vias 4 -> 2
- net MISO: track 48.0 -> 78.6 mm, vias 2 -> 5
- net A1: track 47.3 -> 18.4 mm, vias 5 -> 2
- net D1-TXD: track 26.6 -> 0.00 mm, vias 2 -> 0
- net DTR: track 26.3 -> 0.00 mm, vias 2 -> 0
- net Net-(BT2-Pad2): track 38.8 -> 12.5 mm, vias 0 -> 2
- net NSS: track 46.1 -> 69.8 mm, vias 0 -> 3
- net D0-RXD: track 18.5 -> 0.00 mm, vias 2 -> 0
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
Commit message: routing test 3
Parts:
- C11, R5: moved to F.Cu
- C7: moved to B.Cu
- moved U2 24.1 mm to (157.5, 96.3)
- moved JP3 24.0 mm to (133.6, 95.1), turned to 90 degrees
- moved C4 19.2 mm to (157.2, 93.5), turned to 0 degrees
- moved C11 17.2 mm to (143.7, 96.2), turned to 180 degrees
- moved R5 12.5 mm to (145.4, 89.5), turned to 270 degrees
- moved C10 12.3 mm to (152.3, 82.8), turned to 0 degrees
- moved C9 10.5 mm to (138.7, 80.3), turned to 90 degrees
- moved R2 9.32 mm to (153.7, 93.5), turned to 0 degrees
- moved C7 9.21 mm to (141.2, 82.5)
- moved C8 7.73 mm to (152.4, 80.5), turned to 0 degrees
- moved SW2 3.05 mm to (148.8, 82.0), turned to 180 degrees
- moved J5 1.80 mm to (155.7, 81.5)
- turned U4 to 180 degrees
Routing:
- net VCC: track 218.2 -> 151.6 mm
- net GND: track 98.4 -> 154.0 mm, vias 4 -> 8
- net D3: track 0.00 -> 53.2 mm, vias 0 -> 2
- net D4: track 0.00 -> 44.6 mm, vias 0 -> 4
- net +3.3V: track 23.5 -> 57.6 mm, vias 2 -> 3
- net Net-(C6-Pad1): track 41.7 -> 74.7 mm
- net Ext-Pwr-Sense: track 4.79 -> 37.2 mm, vias 0 -> 3
- net D9: track 91.3 -> 59.7 mm, vias 6 -> 2
- net D1-TXD: track 0.00 -> 28.6 mm, vias 0 -> 2
- net Net-(BT2-Pad2): track 12.5 -> 38.7 mm
- net D0-RXD: track 0.00 -> 26.0 mm, vias 0 -> 2
- net A3: track 27.3 -> 4.64 mm, vias 2 -> 0
- net A0: track 23.6 -> 45.3 mm, vias 2 -> 5
- net SCK: track 62.7 -> 83.5 mm, vias 2 -> 5
- net A1: track 18.4 -> 35.5 mm, vias 2 -> 3
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
Commit message: routing test 4
Parts:
- C11, C4, R2, R5, U2: moved to B.Cu
- C7: moved to F.Cu
- moved C4 24.9 mm to (138.9, 76.6), turned to 90 degrees
- moved D4 24.1 mm to (150.4, 75.2), turned to 270 degrees
- moved U2 23.5 mm to (139.4, 81.3), turned to 90 degrees
- moved D5 21.3 mm to (139.2, 75.2), turned to 270 degrees
- moved D3 20.4 mm to (146.8, 75.2), turned to 270 degrees
- moved C11 19.3 mm to (141.7, 77.0)
- moved R8 19.1 mm to (150.4, 78.7), turned to 270 degrees
- moved R10 17.5 mm to (139.2, 78.7), turned to 270 degrees
- moved C10 17.3 mm to (136.4, 89.7), turned to 90 degrees
- moved D2 16.8 mm to (143.3, 75.2), turned to 270 degrees
- moved R2 16.0 mm to (142.2, 82.3), turned to 270 degrees
- moved R7 15.4 mm to (146.8, 78.7), turned to 270 degrees
- moved C9 14.5 mm to (150.1, 89.2), turned to 0 degrees
- moved R6 12.0 mm to (143.3, 78.7), turned to 270 degrees
- moved C8 10.9 mm to (150.1, 91.2)
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Routing:
- net GND: track 154.0 -> 62.5 mm, vias 8 -> 1
- net Net-(C6-Pad1): track 74.7 -> 10.7 mm, vias 2 -> 0
- net MISO: track 93.1 -> 32.9 mm, vias 5 -> 0
- net Net-(C3-Pad2): track 57.9 -> 0.00 mm, vias 3 -> 0
- net +3.3V: track 57.6 -> 0.00 mm, vias 3 -> 0
- net DTR: track 0.00 -> 50.6 mm, vias 0 -> 5
- net D2: track 55.0 -> 100.8 mm, vias 5 -> 6
- net D4: track 44.6 -> 3.28 mm, vias 4 -> 1
- net Net-(BT2-Pad2): track 38.7 -> 0.00 mm, vias 2 -> 0
- net SCK: track 83.5 -> 48.2 mm, vias 5 -> 4
- net A3: track 4.64 -> 38.5 mm, vias 0 -> 3
- net Ext-Pwr-Sense: track 37.2 -> 4.79 mm, vias 3 -> 0
- net A1: track 35.5 -> 67.4 mm, vias 3 -> 4
- net Net-(BT1-Pad1): track 29.2 -> 0.00 mm, vias 2 -> 0
- net D3: track 53.2 -> 28.4 mm
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
Commit message: routing test 5
Parts:
- C3, JP2, R1, R9: moved to B.Cu
- SW3: footprint switches:Reed-MKA-14103-EXT-SILK -> switches:Reed-MKA-14103
- moved U5 54.4 mm to (186.7, 73.7), turned to 0 degrees
- moved Q1 50.6 mm to (133.9, 95.0), turned to 180 degrees
- moved BT2 48.7 mm to (135.4, 89.4), turned to 0 degrees
- moved BT3 48.5 mm to (183.9, 102.6), turned to 180 degrees
- moved J2 48.0 mm to (136.4, 75.9), turned to 0 degrees
- moved C2 41.1 mm to (134.6, 85.9)
- moved C6 39.6 mm to (138.9, 79.5), turned to 0 degrees
- moved SW3 36.7 mm to (150.4, 82.5), turned to 0 degrees
- moved U3 31.9 mm to (145.3, 77.2), turned to 0 degrees
- moved L1 31.3 mm to (135.6, 94.2), turned to 90 degrees
- moved U1 30.7 mm to (139.2, 85.9)
- moved C3 28.7 mm to (134.1, 98.0), turned to 180 degrees
- moved R3 28.0 mm to (147.6, 82.3), turned to 0 degrees
- moved J5 28.0 mm to (183.9, 81.3)
- moved J3 27.4 mm to (166.9, 77.7), turned to 180 degrees
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Routing:
- net RESET: track 29.8 -> 103.8 mm, vias 1 -> 4
- net +3.3V: track 0.00 -> 69.0 mm, vias 0 -> 3
- net Net-(C3-Pad2): track 0.00 -> 68.2 mm, vias 0 -> 6
- net Net-(BT1-Pad1): track 0.00 -> 57.1 mm, vias 0 -> 4
- net VCC: track 141.0 -> 190.2 mm, vias 13 -> 11
- net D3: track 28.4 -> 76.3 mm, vias 2 -> 5
- net Net-(BT2-Pad2): track 0.00 -> 41.1 mm
- net A0: track 33.7 -> 72.2 mm, vias 2 -> 4
- net MOSI: track 43.0 -> 78.7 mm, vias 0 -> 4
- net Net-(C6-Pad1): track 10.7 -> 45.6 mm, vias 0 -> 2
- net DTR: track 50.6 -> 83.1 mm
- net D4: track 3.28 -> 35.1 mm, vias 1 -> 2
- net NSS: track 39.7 -> 69.1 mm, vias 0 -> 5
- net Net-(C5-Pad1): track 26.6 -> 51.7 mm, vias 2 -> 4
- net D1-TXD: track 17.4 -> 42.1 mm, vias 2 -> 4
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
Commit message: routing test 6
Parts:
- added JP4: 1xAAA, Jumper:SolderJumper-2_P1.3mm_Open_RoundedPad1.0x1.5mm, B.Cu at (185.4, 107.2)
- turned C7 to 180 degrees
Routing:
- net GND: track 80.3 -> 173.7 mm, vias 4 -> 20
- net +3.3V: track 69.0 -> 105.5 mm, vias 3 -> 4
- net Net-(J3-Pad2): track 5.08 -> 39.9 mm, vias 0 -> 2
- net DTR: track 83.1 -> 55.3 mm
- net VCC: track 190.2 -> 205.5 mm, vias 11 -> 12
- net Net-(J2-Pad6): track 0.00 -> 13.5 mm
- net Net-(BT2-Pad2): track 41.1 -> 51.5 mm, vias 0 -> 2
- net Net-(C7-Pad1): track 3.00 -> 9.80 mm, vias 0 -> 2
- net A1: track 46.8 -> 51.8 mm
- net D1-TXD: track 42.1 -> 37.8 mm, vias 4 -> 2
- net D0-RXD: track 30.3 -> 33.8 mm
- net A0: track 72.2 -> 69.4 mm, vias 4 -> 6
- net RESET: track 103.8 -> 102.0 mm
- net A2: track 41.2 -> 40.1 mm
- net Net-(JP2-Pad2): track 20.5 -> 20.9 mm, vias 1 -> 3
- added copper zone on B.Cu, net GND
- added copper zone on F.Cu, net GND

Commit message: finalization 1
Parts:
- added G***: LOGO, logo:d-diot-logo-small, F.Cu at (179.2, 97.0)
- turned C4 to 0 degrees
- turned C7 to 0 degrees
Routing:
- net GND: track 173.7 -> 221.5 mm, vias 20 -> 42
- net A3: track 56.8 -> 46.9 mm, vias 5 -> 3
- net VCC: track 205.5 -> 198.4 mm
- net Net-(C7-Pad1): track 9.80 -> 3.00 mm, vias 2 -> 0
- net Net-(L1-Pad2): track 8.75 -> 12.1 mm
- net DTR: track 55.3 -> 52.2 mm
- net Net-(J3-Pad2): track 39.9 -> 41.5 mm, vias 2 -> 0
- net +3.3V: track 105.5 -> 104.6 mm, vias 4 -> 5
- net MOSI: track 78.7 -> 79.6 mm
Other:
- board text added: "+"
- board text added: "-"

Commit message: Mini-BT-Pcb-328P v.1.0
Other:
- board text added: "3.3V"
- board text added: "A0"
- board text added: "A1"
- board text added: "A2"
- board text added: "A3"
- board text added: "A6"
- board text added: "A7"
- board text added: "ANT"
- board text added: "BT2 1xAAA"
- board text added: "Booster"
- board text added: "CE"
- board text added: "D2"
- board text added: "D3"
- board text added: "D5"
- board text added: "D6"
- board text added: "D9"
- board text added: "DTR"
- board text added: "GND"
- board text added: "MCU-D4"
- board text added: "MISO"
- board text added: "MOSI"
- board text added: "MYSX 2.6"
- board text added: "Mini-BT-Pcb-328P v.1.0"
- board text added: "NSS"
- board text added: "OFF"
- board text added: "ON"
- board text added: "RFM69-RST"
- board text added: "RST"
- board text added: "RXD"
- board text added: "SCK"
- board text added: "SCL"
- board text added: "SDA"
- board text added: "TXD"
- board text added: "VCC"
- board text added: "Vbatt"
- board text added: "Vin"
Changed lines of the file:
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@@
   (general
     (thickness 1.6)
-    (drawings 6)
-    (tracks 931)
+    (drawings 50)
+    (tracks 932)
     (zones 0)
     (modules 53)
@@
     (tags "solder jumper open")
     (attr virtual)
-    (fp_text reference JP2 (at 0.03 1.778 270) (layer B.SilkS)
-      (effects (font (size 1 1) (thickness 0.15)) (justify mirror))
+    (fp_text reference JP2 (at 0.411 -1.651 90) (layer B.SilkS)
+      (effects (font (size 0.7 0.7) (thickness 0.12)) (justify mirror))
     )
     (fp_text value Radio-rst (at 0 -1.9 270) (layer B.Fab)
@@
       (effects (font (size 0.800307 0.800307) (thickness 0.05)) (justify mirror))
     )
-    (fp_text value FDN337N (at -2.032 0.508 270) (layer B.SilkS)
+    (fp_text value FDN337N (at -2.032 0.254 270) (layer B.SilkS)
       (effects (font (size 0.640925 0.640925) (thickness 0.05)) (justify mirror))
     )
@@
     (tags resistor)
     (attr smd)
-    (fp_text reference R1 (at -2.7155 0 270) (layer B.SilkS)
+    (fp_text reference R1 (at 0 -1.651 270) (layer B.SilkS)
       (effects (font (size 1 1) (thickness 0.15)) (justify mirror))
     )
@@
     (tags resistor)
     (attr smd)
-    (fp_text reference R9 (at 2.794 0.254 90) (layer B.SilkS)
+    (fp_text reference R9 (at 0 1.651 270) (layer B.SilkS)
       (effects (font (size 1 1) (thickness 0.15)) (justify mirror))
     )
@@
       (xy -0.339993 3.369811) (xy -0.309687 3.369775) (xy -0.275638 3.369787)) (layer F.SilkS) (width 0.01))
   )
+  (gr_text "MYSX 2.6" (at 143.51 97.028) (layer F.SilkS)
+    (effects (font (size 0.7 0.7) (thickness 0.1)))
+  )
+  (gr_text "BT2\n1xAAA" (at 182.753 106.807 270) (layer B.SilkS)
+    (effects (font (size 0.7 0.7) (thickness 0.1)) (justify mirror))
+  )
+  (gr_text Vin (at 135.89 107.188 270) (layer B.SilkS)
+    (effects (font (size 0.7 0.7) (thickness 0.1)) (justify mirror))
+  )
+  (gr_text GND (at 182.626 97.282) (layer B.SilkS)
+    (effects (font (size 0.7 0.7) (thickness 0.1)) (justify mirror))
+  )
+  (gr_text RFM69-RST (at 180.594 96.012) (layer B.SilkS)
+    (effects (font (size 0.7 0.7) (thickness 0.1)) (justify mirror))
+  )
+  (gr_text D9 (at 183.007 94.742) (layer B.SilkS)
+    (effects (font (size 0.7 0.7) (thickness 0.1)) (justify mirror))
+  )
+  (gr_text - (at 151.638 73.66) (layer B.SilkS)
+    (effects (font (size 0.7 0.7) (thickness 0.1)) (justify mirror))
+  )
+  (gr_text + (at 151.638 78.74) (layer B.SilkS)
+    (effects (font (size 0.7 0.7) (thickness 0.1)) (justify mirror))
+  )
+  (gr_text VCC (at 162.687 76.581) (layer B.SilkS)
+    (effects (font (size 0.7 0.7) (thickness 0.1)) (justify mirror))
+  )
+  (gr_text 3.3V (at 168.148 79.248) (layer B.SilkS)
+    (effects (font (size 0.7 0.7) (thickness 0.1)) (justify mirror))
+  )
+  (gr_text Vbatt (at 168.275 74.041) (layer B.SilkS)
+    (effects (font (size 0.7 0.7) (thickness 0.1)) (justify mirror))
+  )
+  (gr_text ANT (at 185.928 81.28 90) (layer F.SilkS)
+    (effects (font (size 0.7 0.7) (thickness 0.1)))
+  )
+  (gr_text CE (at 163.322 79.121) (layer F.SilkS)
+    (effects (font (size 0.7 0.7) (thickness 0.1)))
+  )
+  (gr_text CE (at 163.322 76.581) (layer F.SilkS)
+    (effects (font (size 0.7 0.7) (thickness 0.1)))
+  )
+  (gr_text CE (at 163.322 74.168) (layer F.SilkS)
+    (effects (font (size 0.7 0.7) (thickness 0.1)))
+  )
+  (gr_text Booster (at 161.798 77.724 90) (layer F.SilkS)
+    (effects (font (size 0.7 0.7) (thickness 0.1)))
+  )
+  (gr_text MCU-D4 (at 171.831 76.581) (layer F.SilkS)
+    (effects (font (size 0.7 0.7) (thickness 0.1)))
+  )
+  (gr_text OFF (at 170.688 81.661) (layer F.SilkS)
+    (effects (font (size 0.7 0.7) (thickness 0.1)))
+  )
+  (gr_text ON (at 170.434 74.041) (layer F.SilkS)
+    (effects (font (size 0.7 0.7) (thickness 0.1)))
+  )
+  (gr_text A7 (at 164.719 86.995) (layer F.SilkS)
+    (effects (font (size 0.7 0.7) (thickness 0.1)))
+  )
+  (gr_text A6 (at 169.291 92.075) (layer F.SilkS)
+    (effects (font (size 0.7 0.7) (thickness 0.1)))
+  )
+  (gr_text A3 (at 158.115 98.933 90) (layer F.SilkS)
+    (effects (font (size 0.7 0.7) (thickness 0.1)))
+  )
+  (gr_text A2 (at 158.115 106.045 90) (layer F.SilkS)
+    (effects (font (size 0.7 0.7) (thickness 0.1)))
+  )
+  (gr_text NSS (at 155.575 98.552 90) (layer F.SilkS)
+    (effects (font (size 0.7 0.7) (thickness 0.1)))
+  )
+  (gr_text SCK (at 155.575 106.426 90) (layer F.SilkS)
+    (effects (font (size 0.7 0.7) (thickness 0.1)))
+  )
+  (gr_text MOSI (at 153.162 106.68 90) (layer F.SilkS)
+    (effects (font (size 0.7 0.7) (thickness 0.1)))
+  )
+  (gr_text MISO (at 152.908 98.552 90) (layer F.SilkS)
+    (effects (font (size 0.7 0.7) (thickness 0.1)))
+  )
+  (gr_text A0 (at 150.495 106.045 90) (layer F.SilkS)
+    (effects (font (size 0.7 0.7) (thickness 0.1)))
+  )
+  (gr_text A1 (at 150.495 98.933 90) (layer F.SilkS)
+    (effects (font (size 0.7 0.7) (thickness 0.1)))
+  )
+  (gr_text SCL (at 147.955 106.426 90) (layer F.SilkS)
+    (effects (font (size 0.7 0.7) (thickness 0.1)))
+  )
+  (gr_text SDA (at 147.955 98.806 90) (layer F.SilkS)
+    (effects (font (size 0.7 0.7) (thickness 0.1)))
+  )
+  (gr_text D5 (at 145.415 106.045 90) (layer F.SilkS)
+    (effects (font (size 0.7 0.7) (thickness 0.1)))
+  )
+  (gr_text D6 (at 145.415 99.06 90) (layer F.SilkS)
+    (effects (font (size 0.7 0.7) (thickness 0.1)))
+  )
+  (gr_text D2 (at 142.875 106.299 90) (layer F.SilkS)
+    (effects (font (size 0.7 0.7) (thickness 0.1)))
+  )
+  (gr_text D3 (at 142.875 99.06 90) (layer F.SilkS)
+    (effects (font (size 0.7 0.7) (thickness 0.1)))
+  )
+  (gr_text RST (at 140.335 106.426 90) (layer F.SilkS)
+    (effects (font (size 0.7 0.7) (thickness 0.1)))
+  )
+  (gr_text DTR (at 140.335 98.806 90) (layer F.SilkS)
+    (effects (font (size 0.7 0.7) (thickness 0.1)))
+  )
+  (gr_text TXD (at 137.795 106.426 90) (layer F.SilkS)
+    (effects (font (size 0.7 0.7) (thickness 0.1)))
+  )
+  (gr_text RXD (at 137.795 98.806 90) (layer F.SilkS)
+    (effects (font (size 0.7 0.7) (thickness 0.1)))
+  )
+  (gr_text GND (at 135.255 98.806 90) (layer F.SilkS)
+    (effects (font (size 0.7 0.7) (thickness 0.1)))
+  )
+  (gr_text VCC (at 135.255 106.426 90) (layer F.SilkS)
+    (effects (font (size 0.7 0.7) (thickness 0.1)))
+  )
+  (gr_text Vin (at 132.588 106.172 90) (layer F.SilkS)
+    (effects (font (size 0.7 0.7) (thickness 0.1)))
+  )
+  (gr_text 3.3V (at 132.715 98.679 90) (layer F.SilkS)
+    (effects (font (size 0.7 0.7) (thickness 0.1)))
+  )
+  (gr_text "Mini-BT-Pcb-328P v.1.0" (at 158.623 96.012) (layer F.SilkS)
+    (effects (font (size 1.2 1.2) (thickness 0.2)))
+  )
   (gr_text - (at 176.657 96.012) (layer B.SilkS)
     (effects (font (size 1.5 1.5) (thickness 0.3)) (justify mirror))
@@
   (segment (start 183.134 97.282) (end 184.912 97.282) (width 0.16) (layer B.Cu) (net 9) (status 20))
   (segment (start 161.544 81.374) (end 161.544 81.2015) (width 0.16) (layer B.Cu) (net 9) (status 30))
-  (segment (start 160.368 82.55) (end 161.544 81.374) (width 0.16) (layer B.Cu) (net 9) (status 30))
   (segment (start 139.8755 79.502) (end 139.7 79.502) (width 0.3) (layer B.Cu) (net 9) (status 30))
   (segment (start 152.588 79.926) (end 152.588 79.726) (width 0.16) (layer B.Cu) (net 9) (status 30))
@@
   (segment (start 133.684999 87.244595) (end 133.684999 87.136783) (width 0.16) (layer F.Cu) (net 9))
   (via (at 133.858 91.694) (size 0.65) (drill 0.35) (layers F.Cu B.Cu) (net 9))
+  (segment (start 160.368 82.3775) (end 161.544 81.2015) (width 0.3) (layer B.Cu) (net 9))
+  (segment (start 160.368 82.55) (end 160.368 82.3775) (width 0.3) (layer B.Cu) (net 9))
   (segment (start 183.958 81.342) (end 183.896 81.28) (width 1.3) (layer F.Cu) (net 10) (status 30))
   (segment (start 183.958 85.344) (end 183.958 81.342) (width 1.3) (layer F.Cu) (net 10) (status 30))
