File: Mini-BT-Pcb-328P.kicad_pcb (KiCad board)
At the start: 2 copper layers, 55 x 35 mm, 53 parts, among them J1 Analog IN, J2 USB_B_Micro, J3 Booster CE, J5 ANT, P1 MYSX_2.6, Q1 FDN338P, Q2 FDN337N, SW2 Reset, SW3 SW_Reed, U1 ME2188C33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

Commit message: version 2.0
Parts:
- added JP5: Jumper_2_Open, Jumper:SolderJumper-2_P1.3mm_Open_RoundedPad1.0x1.5mm, F.Cu at (164.3, 93.2)
Routing:
- net Net-(BT1-Pad1): track 57.1 -> 61.9 mm
- net A7: track 12.9 -> 17.7 mm
Other:
- board text added: "Mini-BT-Pcb-328P v.2.0"
- board text removed: "Mini-BT-Pcb-328P v.1.0"
Changed lines of the file:
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@@
   (general
     (thickness 1.6)
-    (drawings 50)
-    (tracks 932)
+    (drawings 52)
+    (tracks 940)
     (zones 0)
-    (modules 53)
+    (modules 54)
     (nets 58)
   )
@@
   (title_block
     (title Mini-BT-Pcb-328P)
-    (date 2019-10-11)
-    (rev 1.0)
+    (date 2020-02-09)
+    (rev 2.0)
     (company d-diot)
     (comment 1 info@d-diot.com)
@@
   )
   (setup
-    (last_trace_width 0.3)
+    (last_trace_width 0.16)
     (user_trace_width 0.3)
     (user_trace_width 1.3)
@@
       (drillshape 0)
       (scaleselection 1)
-      (outputdirectory "export/gerber/v.1.0/"))
+      (outputdirectory "export/gerber/v.2.0/"))
   )
   (net 0 "")
@@
     (add_net Vin)
   )
+  (module Jumper:SolderJumper-2_P1.3mm_Open_RoundedPad1.0x1.5mm (layer F.Cu)
+    (at 164.338 93.218 270)
+    (descr "SMD Solder Jumper, 1x1.5mm, rounded Pads, 0.3mm gap, open")
+    (tags "solder jumper open")
+    (attr virtual)
+    (fp_text reference JP5 (at 0 1.778 270) (layer F.SilkS)
+      (effects (font (size 0.8 0.8) (thickness 0.12)))
+    )
+    (fp_text value Jumper_2_Open (at 0 1.9 270) (layer F.Fab)
+      (effects (font (size 1 1) (thickness 0.15)))
+    )
+    (fp_arc (start 0.7 -0.3) (end 1.4 -0.3) (angle -90) (layer F.SilkS) (width 0.12))
+    (fp_arc (start 0.7 0.3) (end 0.7 1) (angle -90) (layer F.SilkS) (width 0.12))
+    (fp_arc (start -0.7 0.3) (end -1.4 0.3) (angle -90) (layer F.SilkS) (width 0.12))
+    (fp_arc (start -0.7 -0.3) (end -0.7 -1) (angle -90) (layer F.SilkS) (width 0.12))
+    (fp_line (start -1.4 0.3) (end -1.4 -0.3) (layer F.SilkS) (width 0.12))
+    (fp_line (start 0.7 1) (end -0.7 1) (layer F.SilkS) (width 0.12))
+    (fp_line (start 1.4 -0.3) (end 1.4 0.3) (layer F.SilkS) (width 0.12))
+    (fp_line (start -0.7 -1) (end 0.7 -1) (layer F.SilkS) (width 0.12))
+    (fp_line (start -1.65 -1.25) (end 1.65 -1.25) (layer F.CrtYd) (width 0.05))
+    (fp_line (start -1.65 -1.25) (end -1.65 1.25) (layer F.CrtYd) (width 0.05))
+    (fp_line (start 1.65 1.25) (end 1.65 -1.25) (layer F.CrtYd) (width 0.05))
+    (fp_line (start 1.65 1.25) (end -1.65 1.25) (layer F.CrtYd) (width 0.05))
+    (pad 1 smd custom (at -0.65 0 270) (size 1 0.5) (layers F.Cu F.Mask)
+      (net 40 A7) (zone_connect 0)
+      (options (clearance outline) (anchor rect))
+      (primitives
+        (gr_circle (center 0 0.25) (end 0.5 0.25) (width 0))
+        (gr_circle (center 0 -0.25) (end 0.5 -0.25) (width 0))
+        (gr_poly (pts
+           (xy 0 -0.75) (xy 0.5 -0.75) (xy 0.5 0.75) (xy 0 0.75)) (width 0))
+      ))
+    (pad 2 smd custom (at 0.65 0 270) (size 1 0.5) (layers F.Cu F.Mask)
+      (net 18 "Net-(BT1-Pad1)") (zone_connect 0)
+      (options (clearance outline) (anchor rect))
+      (primitives
+        (gr_circle (center 0 0.25) (end 0.5 0.25) (width 0))
+        (gr_circle (center 0 -0.25) (end 0.5 -0.25) (width 0))
+        (gr_poly (pts
+           (xy 0 -0.75) (xy -0.5 -0.75) (xy -0.5 0.75) (xy 0 0.75)) (width 0))
+      ))
+  )
   (module Resistor_SMD:R_0805_2012Metric (layer F.Cu)
     (at 148.082 79.1695 270)
@@
     (tags "Surface mounted pin header SMD 1x02 2.54mm single row style1 pin1 left")
     (attr smd)
-    (fp_text reference J1 (at 0.508 -1.524 270) (layer F.SilkS)
+    (fp_text reference J1 (at -2.286 1.778 270) (layer F.SilkS)
       (effects (font (size 1 1) (thickness 0.15)))
     )
@@
     (pad 1 np_thru_hole circle (at 0 0) (size 2.5 2.5) (drill 2.5) (layers *.Cu *.Mask))
   )
-  (module logo:d-diot-logo-small (layer F.Cu)
+  (module logo:d-diot-logo-small locked (layer F.Cu)
     (at 179.197 97.028)
     (fp_text reference G*** (at 0 0) (layer F.SilkS) hide
@@
       (xy -0.339993 3.369811) (xy -0.309687 3.369775) (xy -0.275638 3.369787)) (layer F.SilkS) (width 0.01))
   )
+  (gr_text Vbatt (at 167.132 93.98) (layer F.SilkS)
+    (effects (font (size 0.7 0.7) (thickness 0.1)))
+  )
+  (gr_text A7 (at 166.37 92.71) (layer F.SilkS)
+    (effects (font (size 0.7 0.7) (thickness 0.1)))
+  )
   (gr_text "MYSX 2.6" (at 143.51 97.028) (layer F.SilkS)
     (effects (font (size 0.7 0.7) (thickness 0.1)))
@@
     (effects (font (size 0.7 0.7) (thickness 0.1)))
   )
-  (gr_text "Mini-BT-Pcb-328P v.1.0" (at 158.623 96.012) (layer F.SilkS)
+  (gr_text "Mini-BT-Pcb-328P v.2.0" (at 158.623 96.012) (layer F.SilkS)
     (effects (font (size 1.2 1.2) (thickness 0.2)))
   )
@@
   (segment (start 138.6055 81.6125) (end 138.710001 81.507999) (width 0.16) (layer B.Cu) (net 8) (status 30))
   (segment (start 138.6055 82.042) (end 138.6055 81.6125) (width 0.16) (layer B.Cu) (net 8) (status 30))
-  (segment (start 133.162 84.8235) (end 133.1745 84.836) (width 0.16) (layer B.Cu) (net 9) (status 30))
   (segment (start 143.8425 90.17) (end 145.172999 91.500499) (width 0.3) (layer F.Cu) (net 8) (status 10))
   (segment (start 136.413 105.156) (end 136.398 105.141) (width 0.3) (layer F.Cu) (net 8) (status 30))
@@
   (segment (start 133.162 82.9485) (end 133.162 82.526) (width 0.16) (layer B.Cu) (net 8))
   (segment (start 135.0495 84.836) (end 133.162 82.9485) (width 0.16) (layer B.Cu) (net 8))
+  (segment (start 133.162 84.8235) (end 133.1745 84.836) (width 0.16) (layer B.Cu) (net 9) (status 30))
   (segment (start 185.958 83.684) (end 185.958 85.344) (width 0.16) (layer F.Cu) (net 9) (status 20))
   (segment (start 186.309601 83.332399) (end 185.958 83.684) (width 0.16) (layer F.Cu) (net 9))
@@
   (segment (start 163.068 104.134) (end 163.062 104.14) (width 0.3) (layer F.Cu) (net 18) (status 30))
   (via (at 163.068 96.266) (size 0.65) (drill 0.35) (layers F.Cu B.Cu) (net 18))
-  (segment (start 163.062 104.14) (end 163.062 96.272) (width 0.3) (layer F.Cu) (net 18) (status 10))
   (segment (start 163.062 96.272) (end 163.068 96.266) (width 0.3) (layer F.Cu) (net 18))
   (segment (start 163.068 96.266) (end 144.9 96.266) (width 0.3) (layer B.Cu) (net 18) (status 20))
@@
   (segment (start 140.378 93.896) (end 140.462 93.98) (width 0.3) (layer B.Cu) (net 18))
   (segment (start 140.462 93.98) (end 140.462 96.266) (width 0.3) (layer F.Cu) (net 18))
+  (segment (start 163.709444 97.79) (end 163.062 97.79) (width 0.16) (layer F.Cu) (net 18))
+  (segment (start 164.342001 97.157443) (end 163.709444 97.79) (width 0.16) (layer F.Cu) (net 18))
+  (segment (start 164.342001 94.472001) (end 164.342001 97.157443) (width 0.16) (layer F.Cu) (net 18))
+  (segment (start 164.338 94.468) (end 164.342001 94.472001) (width 0.16) (layer F.Cu) (net 18))
+  (segment (start 164.338 93.868) (end 164.338 94.468) (width 0.16) (layer F.Cu) (net 18))
+  (segment (start 163.062 97.79) (end 163.062 96.272) (width 0.3) (layer F.Cu) (net 18))
+  (segment (start 163.062 104.14) (end 163.062 97.79) (width 0.3) (layer F.Cu) (net 18))
   (segment (start 183.896 101.146) (end 183.896 102.616) (width 0.3) (layer B.Cu) (net 19) (status 20))
   (segment (start 186.01201 99.02999) (end 183.896 101.146) (width 0.3) (layer B.Cu) (net 19))
@@
   (segment (start 163.479 88.235) (end 163.576 88.138) (width 0.16) (layer B.Cu) (net 40))
   (segment (start 163.576 88.138) (end 165.477 88.138) (width 0.16) (layer F.Cu) (net 40) (status 20))
+  (segment (start 164.338 88.9) (end 163.576 88.138) (width 0.16) (layer F.Cu) (net 40))
+  (segment (start 164.338 92.568) (end 164.338 88.9) (width 0.16) (layer F.Cu) (net 40))
   (via (at 167.553 85.441) (size 0.65) (drill 0.35) (layers F.Cu B.Cu) (net 41))
   (segment (start 167.456 85.344) (end 167.553 85.441) (width 0.16) (layer B.Cu) (net 41))
