File: Mini-BT-Pcb-328P.sch (KiCad schematic (older format))
At the start: 50 parts, among them J1 Analog IN, J2 USB_B_Micro, J5 ANT, J6 Booster, P1 MYSX_2.6, Q1 FDN338P, Q2 FDN337N, SW2 Reset, SW3 SW_Reed, U1 ME2188C33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

Commit message: routing test 2
Parts:
- removed J6: Booster, Connector_PinHeader_2.54mm:PinHeader_2x03_P2.54mm_Vertical_SMD, symbol Connector_Generic:Conn_02x03_Top_Bottom
- added J3: Booster CE, Connector_PinHeader_2.54mm:PinHeader_2x03_P2.54mm_Vertical_SMD, symbol Connector_Generic:Conn_02x03_Odd_Even
Connections:
- net D4: now also J3.3 (Pin_3)
- net at U1.1 (CE): now also J3.2 (Pin_2), J3.4 (Pin_4), J3.6 (Pin_6)
- net at R1.1: now also J3.5 (Pin_5)
- net at R9.2: now also J3.1 (Pin_1)
Changed lines of the file:
@@
 Wire Wire Line
 	1500 4900 1750 4900
-$Comp
-L Connector_Generic:Conn_02x03_Top_Bottom J6
-U 1 1 5D944FEC
-P 900 4050
-F 0 "J6" H 950 4367 50  0000 C CNN
-F 1 "Booster" H 950 4276 50  0000 C CNN
-F 2 "Connector_PinHeader_2.54mm:PinHeader_2x03_P2.54mm_Vertical_SMD" H 900 4050 50  0001 C CNN
-F 3 "~" H 900 4050 50  0001 C CNN
-	1    900  4050
-	1    0    0    -1
-$EndComp
 Wire Wire Line
 	1200 4050 1400 4050
@@
 Wire Wire Line
 	3050 6850 3200 6850
+$Comp
+L Connector_Generic:Conn_02x03_Odd_Even J3
+U 1 1 5D99E722
+P 900 4050
+F 0 "J3" H 950 4367 50  0000 C CNN
+F 1 "Booster CE" H 950 4276 50  0000 C CNN
+F 2 "Connector_PinHeader_2.54mm:PinHeader_2x03_P2.54mm_Vertical_SMD" H 900 4050 50  0001 C CNN
+F 3 "~" H 900 4050 50  0001 C CNN
+	1    900  4050
+	1    0    0    -1
+$EndComp
 $EndSCHEMATC

Commit message: routing test 5
Parts:
- SW3: footprint switches:Reed-MKA-14103-EXT-SILK -> switches:Reed-MKA-14103
Changed lines of the file:
@@
 F 0 "SW3" V 3354 2685 50  0000 L CNN
 F 1 "SW_Reed" V 3445 2685 50  0000 L CNN
-F 2 "switches:Reed-MKA-14103-EXT-SILK" H 3400 2600 50  0001 C CNN
+F 2 "switches:Reed-MKA-14103" H 3400 2600 50  0001 C CNN
 F 3 "" H 3400 2600 50  0001 C CNN
 	1    3400 2600

Commit message: routing test 6
Parts:
- added JP4: 1xAAA, Jumper:SolderJumper-2_P1.3mm_Open_RoundedPad1.0x1.5mm, symbol Jumper:Jumper_2_Open
Connections:
- net GND: now also JP4.2 (B)
- net at BT2.2 (-), BT3.1 (+): now also JP4.1 (A)
Changed lines of the file:
@@
+	1    0    0    -1
+$EndComp
+$Comp
+L Jumper:Jumper_2_Open JP4
+U 1 1 5D9FB1BA
+P 1550 7100
+F 0 "JP4" V 1504 7198 50  0000 L CNN
+F 1 "1xAAA" V 1595 7198 50  0000 L CNN
+F 2 "Jumper:SolderJumper-2_P1.3mm_Open_RoundedPad1.0x1.5mm" H 1550 7100 50  0001 C CNN
+F 3 "~" H 1550 7100 50  0001 C CNN
+	1    1550 7100
+	0    1    1    0
+$EndComp
+Wire Wire Line
+	1750 6200 1550 6200
+Wire Wire Line
+	1550 6200 1550 6900
+Connection ~ 1750 6200
+$Comp
+L power:GND #PWR02
+U 1 1 5D9FD7B0
+P 1550 7300
+F 0 "#PWR02" H 1550 7050 50  0001 C CNN
+F 1 "GND" H 1555 7127 50  0000 C CNN
+F 2 "" H 1550 7300 50  0001 C CNN
+F 3 "" H 1550 7300 50  0001 C CNN
+	1    1550 7300
 	1    0    0    -1
 $EndComp

Commit message: version 2.0
Parts:
- added JP5: Jumper_2_Open, Jumper:SolderJumper-2_P1.3mm_Open_RoundedPad1.0x1.5mm, symbol Jumper:Jumper_2_Open
Connections:
- net A7: now also JP5.1 (A)
- net at BT1.1 (+), BT2.1 (+), C1.1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: now also JP5.2 (B)
Changed lines of the file:
@@
 Sheet 1 1
 Title "Mini-BT-Pcb-328P"
-Date "2019-10-05"
-Rev "1.0"
+Date "2020-02-09"
+Rev "2.0"
 Comp "d-diot"
 Comment1 "Author: Francesco Berghi"
@@
 	1    0    0    -1
 $EndComp
-Wire Wire Line
-	1750 4900 1750 5300
 $Comp
 L Device:R R9
@@
 	1    0    0    -1
 $EndComp
+$Comp
+L Jumper:Jumper_2_Open JP5
+U 1 1 5E406A60
+P 2150 7000
+F 0 "JP5" V 2196 6912 50  0000 R CNN
+F 1 "Jumper_2_Open" V 2105 6912 50  0000 R CNN
+F 2 "Jumper:SolderJumper-2_P1.3mm_Open_RoundedPad1.0x1.5mm" H 2150 7000 50  0001 C CNN
+F 3 "~" H 2150 7000 50  0001 C CNN
+	1    2150 7000
+	0    -1   -1   0
+$EndComp
+Text GLabel 2150 7200 3    50   Input ~ 0
+A7
+Wire Wire Line
+	1750 4900 1750 5300
+Wire Wire Line
+	2150 6800 2150 5800
+Wire Wire Line
+	2150 5800 1750 5800
 $EndSCHEMATC
